File: Disarmed/Analog_Panel.sch (KiCad schematic (older format))
At the start: 24 parts, among them J1 Conn_02x03_Odd_Even, J10 Conn_01x03, J11 Conn_01x03, J12 Conn_01x03, J13 Conn_01x03, J14 Conn_01x02, J15 Conn_01x02, J2 Conn_01x02_Male, J3 Conn_01x03, J4 Conn_01x03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

Commit message: Add new boards
Other:
- note added: "Implements a second I2C interface in software to drive the MAX11616 and MCP47CXBXX"
- note removed: "Drives shift registers via SPI like protocol using SPI hardware (or software transfer)"
- moved on the sheet: U3
Changed lines of the file:
@@
 $Descr A4 11693 8268
 encoding utf-8
-Sheet 1 1
+Sheet 5 6
 Title ""
 Date ""
@@
 AR Path="/6008A670/600EA4F5" Ref="U?"  Part="1"
 AR Path="/600EA4F5" Ref="U1"  Part="1"
-F 0 "U1" H 2728 5728 60  0000 L CNN
+F 0 "U?" H 2728 5728 60  0000 L CNN
 F 1 "ATTINY85-20PU" H 2728 5622 60  0000 L CNN
 F 2 "digikey-footprints:DIP-8_W7.62mm" H 2700 5925 60  0001 L CNN
@@
 AR Path="/6008A670/600EA4FB" Ref="J?"  Part="1"
 AR Path="/600EA4FB" Ref="J1"  Part="1"
-F 0 "J1" H 2550 4642 50  0000 C CNN
+F 0 "J?" H 2550 4642 50  0000 C CNN
 F 1 "Conn_02x03_Odd_Even" H 2550 4551 50  0000 C CNN
 F 2 "Connector_PinHeader_2.54mm:PinHeader_2x03_P2.54mm_Vertical" H 2500 4325 50  0001 C CNN
@@
 AR Path="/6008A670/600EA50F" Ref="C?"  Part="1"
 AR Path="/600EA50F" Ref="C1"  Part="1"
-F 0 "C1" H 3315 5321 50  0000 L CNN
+F 0 "C?" H 3315 5321 50  0000 L CNN
 F 1 "0.1uF" H 3315 5230 50  0000 L CNN
 F 2 "Capacitor_SMD:C_1812_4532Metric_Pad1.57x3.40mm_HandSolder" H 3238 5125 50  0001 C CNN
@@
 AR Path="/6008A670/600EA523" Ref="R?"  Part="1"
 AR Path="/600EA523" Ref="R1"  Part="1"
-F 0 "R1" H 1870 6271 50  0000 L CNN
+F 0 "R?" H 1870 6271 50  0000 L CNN
 F 1 "10K" H 1870 6180 50  0000 L CNN
 F 2 "Resistor_SMD:R_1210_3225Metric_Pad1.30x2.65mm_HandSolder" V 1730 6225 50  0001 C CNN
@@
 AR Path="/6008A670/600EA537" Ref="#PWR?"  Part="1"
 AR Path="/600EA537" Ref="#PWR01"  Part="1"
-F 0 "#PWR01" H 1650 6825 50  0001 C CNN
+F 0 "#PWR?" H 1650 6825 50  0001 C CNN
 F 1 "GND" H 1655 6902 50  0000 C CNN
 F 2 "" H 1650 7075 50  0001 C CNN
@@
 AR Path="/6008A670/600EA53F" Ref="#PWR?"  Part="1"
 AR Path="/600EA53F" Ref="#PWR02"  Part="1"
-F 0 "#PWR02" H 2100 6675 50  0001 C CNN
+F 0 "#PWR?" H 2100 6675 50  0001 C CNN
 F 1 "+5V" H 2115 6998 50  0000 C CNN
 F 2 "" H 2100 6825 50  0001 C CNN
@@
 AR Path="/6008A670/600EA547" Ref="J?"  Part="1"
 AR Path="/600EA547" Ref="J2"  Part="1"
-F 0 "J2" H 2858 7056 50  0000 C CNN
+F 0 "J?" H 2858 7056 50  0000 C CNN
 F 1 "Conn_01x02_Male" H 2858 6965 50  0000 C CNN
 F 2 "Connector_PinHeader_2.54mm:PinHeader_1x02_P2.54mm_Vertical" H 2750 6875 50  0001 C CNN
@@
 AR Path="/6008A670/600EA551" Ref="#FLG?"  Part="1"
 AR Path="/600EA551" Ref="#FLG01"  Part="1"
-F 0 "#FLG01" H 2650 7450 50  0001 C CNN
+F 0 "#FLG?" H 2650 7450 50  0001 C CNN
 F 1 "PWR_FLAG" H 2650 7548 50  0000 C CNN
 F 2 "" H 2650 7375 50  0001 C CNN
@@
 AR Path="/6008A670/600EA559" Ref="#FLG?"  Part="1"
 AR Path="/600EA559" Ref="#FLG02"  Part="1"
-F 0 "#FLG02" H 2650 7700 50  0001 C CNN
+F 0 "#FLG?" H 2650 7700 50  0001 C CNN
 F 1 "PWR_FLAG" H 2650 7798 50  0000 C CNN
 F 2 "" H 2650 7625 50  0001 C CNN
@@
 Implements a I2C interface to the master system.
 Text Notes 650  4725 0    50   ~ 0
-Drives shift registers via SPI like protocol using SPI hardware (or software transfer)
+Implements a second I2C interface in software to drive the MAX11616 and MCP47CXBXX
 Text Notes 800  4825 0    50   ~ 0
 ISP used for programming, shares pins with master system I2C
@@
 L DisarmedParts:MCP47CXBXX U3
 U 1 1 601C1442
-P 4950 4950
-F 0 "U3" H 4925 5565 50  0000 C CNN
-F 1 "MCP47CXBXX" H 4925 5474 50  0000 C CNN
-F 2 "Package_SO:MSOP-10-1EP_3x3mm_P0.5mm_EP1.68x1.88mm_ThermalVias" H 4950 4600 50  0001 C CNN
-F 3 "" H 4950 4600 50  0001 C CNN
-	1    4950 4950
-	1    0    0    -1
-$EndComp
-Wire Wire Line
-	5400 4600 5825 4600
-Wire Wire Line
-	5400 4700 5825 4700
-Wire Wire Line
-	5400 4800 5825 4800
-Wire Wire Line
-	4450 4700 4075 4700
-Wire Wire Line
-	4450 4800 4075 4800
-Wire Wire Line
-	4450 4900 4075 4900
-Wire Wire Line
-	4450 5000 4075 5000
-Wire Wire Line
-	5400 4900 5825 4900
-Wire Wire Line
-	5400 5000 5825 5000
-Wire Wire Line
-	4450 4600 4075 4600
-Text Label 4075 4600 0    50   ~ 0
-VCC
-Text Label 5825 4900 0    50   ~ 0
-GND
-Text Label 4075 4900 0    50   ~ 0
+P 5300 4950
+F 0 "U3" H 5275 5565 50  0000 C CNN
+F 1 "MCP47CXBXX" H 5275 5474 50  0000 C CNN
+F 2 "Package_SO:MSOP-10-1EP_3x3mm_P0.5mm_EP1.68x1.88mm_ThermalVias" H 5300 4600 50  0001 C CNN
+F 3 "" H 5300 4600 50  0001 C CNN
+	1    5300 4950
+	1    0    0    -1
+$EndComp
+Wire Wire Line
+	5750 4600 6175 4600
+Wire Wire Line
+	5750 4700 6175 4700
+Wire Wire Line
+	5750 4800 6175 4800
+Wire Wire Line
+	4800 4700 4425 4700
+Wire Wire Line
+	4800 4800 4425 4800
+Wire Wire Line
+	4800 4900 4425 4900
+Wire Wire Line
+	4800 5000 4425 5000
+Wire Wire Line
+	5750 4900 6175 4900
+Wire Wire Line
+	5750 5000 6175 5000
+Wire Wire Line
+	4800 4600 4425 4600
+Text Label 4425 4600 0    50   ~ 0
+VCC
+Text Label 6175 4900 0    50   ~ 0
+GND
+Text Label 4425 4900 0    50   ~ 0
 AOUT0
-Text Label 4075 5000 0    50   ~ 0
+Text Label 4425 5000 0    50   ~ 0
 AOUT1
-Text Label 4075 4800 0    50   ~ 0
-VCC
-Text Label 4075 4700 0    50   ~ 0
-GND
-Text Label 5825 4800 0    50   ~ 0
-GND
-Text Label 5825 4600 0    50   ~ 0
+Text Label 4425 4800 0    50   ~ 0
+VCC
+Text Label 4425 4700 0    50   ~ 0
+GND
+Text Label 6175 4800 0    50   ~ 0
+GND
+Text Label 6175 4600 0    50   ~ 0
 SDA1
-Text Label 5825 4700 0    50   ~ 0
+Text Label 6175 4700 0    50   ~ 0
 SCL1
-NoConn ~ 5825 5000
+NoConn ~ 6175 5000
 $Comp
 L Connector_Generic:Conn_01x02 J14
