File: Disarmed/SSD_Panel.sch (KiCad schematic (older format))
At the start: 15 parts, among them J1 Conn_02x04_Counter_Clockwise, U1 MAX7219, U2 MCP41010, U3 MAX7219, U4 MAX7219, U5 MAX7219

Commit message: Footprint update to standard PDIP
Parts:
- U2: footprint Package_DIP:DIP-8-16_W7.62mm -> Package_DIP:DIP-8_W7.62mm
Changed lines of the file:
@@
 F 0 "U2" H 1400 1781 50  0000 C CNN
 F 1 "MCP41010" H 1400 1690 50  0000 C CNN
-F 2 "Package_DIP:DIP-8-16_W7.62mm" H 1400 1200 50  0001 C CNN
+F 2 "Package_DIP:DIP-8_W7.62mm" H 1400 1200 50  0001 C CNN
 F 3 "http://ww1.microchip.com/downloads/en/DeviceDoc/11195c.pdf" H 1400 1200 50  0001 C CNN
 	1    1400 1200

Commit message: Add LED Panel
Parts:
- renumbered DS3 to DS2, DS5 to DS3, DS7 to DS4, DS2 to DS5, DS4 to DS6, DS6 to DS7, U2 to U1, U1 to U2
Connections:
- net labels added: +5V
- wire segments 205 -> 209
Changed lines of the file:
@@
 $Descr A4 11693 8268
 encoding utf-8
-Sheet 2 2
+Sheet 2 3
 Title ""
 Date ""
@@
 $EndComp
 $Comp
-L DisarmedParts:D8014CD DS2
+L DisarmedParts:D8014CD DS5
 U 1 1 5FDB2B9D
 P 2800 5350
-F 0 "DS2" V 2285 5000 50  0000 C CNN
+F 0 "DS5" V 2285 5000 50  0000 C CNN
 F 1 "D8014CD" V 2376 5000 50  0000 C CNN
 F 2 "Disarmed:D8041CD" H 2800 5850 50  0001 C CNN
@@
 $EndComp
 $Comp
-L Driver_LED:MAX7219 U1
+L Driver_LED:MAX7219 U2
 U 1 1 5FDAA591
 P 1300 3900
-F 0 "U1" H 1300 5081 50  0000 C CNN
+F 0 "U2" H 1300 5081 50  0000 C CNN
 F 1 "MAX7219" H 1300 4990 50  0000 C CNN
 F 2 "Package_DIP:DIP-24_W7.62mm" H 1250 3950 50  0001 C CNN
@@
 $EndComp
 $Comp
-L DisarmedParts:D8014CD DS3
+L DisarmedParts:D8014CD DS2
 U 1 1 5FDF6F92
 P 5300 2350
-F 0 "DS3" V 4785 2000 50  0000 C CNN
+F 0 "DS2" V 4785 2000 50  0000 C CNN
 F 1 "D8014CD" V 4876 2000 50  0000 C CNN
 F 2 "Disarmed:D8041CD" H 5300 2850 50  0001 C CNN
@@
 $EndComp
 $Comp
-L DisarmedParts:D8014CD DS4
+L DisarmedParts:D8014CD DS6
 U 1 1 5FDF6F98
 P 5300 5350
-F 0 "DS4" V 4785 5000 50  0000 C CNN
+F 0 "DS6" V 4785 5000 50  0000 C CNN
 F 1 "D8014CD" V 4876 5000 50  0000 C CNN
 F 2 "Disarmed:D8041CD" H 5300 5850 50  0001 C CNN
@@
 $EndComp
 $Comp
-L DisarmedParts:D8014CD DS5
+L DisarmedParts:D8014CD DS3
 U 1 1 5FDF8DD1
 P 7800 2350
-F 0 "DS5" V 7285 2000 50  0000 C CNN
+F 0 "DS3" V 7285 2000 50  0000 C CNN
 F 1 "D8014CD" V 7376 2000 50  0000 C CNN
 F 2 "Disarmed:D8041CD" H 7800 2850 50  0001 C CNN
@@
 $EndComp
 $Comp
-L DisarmedParts:D8014CD DS6
+L DisarmedParts:D8014CD DS7
 U 1 1 5FDF8DD7
 P 7800 5350
-F 0 "DS6" V 7285 5000 50  0000 C CNN
+F 0 "DS7" V 7285 5000 50  0000 C CNN
 F 1 "D8014CD" V 7376 5000 50  0000 C CNN
 F 2 "Disarmed:D8041CD" H 7800 5850 50  0001 C CNN
@@
 $EndComp
 $Comp
-L DisarmedParts:D8014CD DS7
+L DisarmedParts:D8014CD DS4
 U 1 1 5FDFC2C0
 P 10300 2350
-F 0 "DS7" V 9785 2000 50  0000 C CNN
+F 0 "DS4" V 9785 2000 50  0000 C CNN
 F 1 "D8014CD" V 9876 2000 50  0000 C CNN
 F 2 "Disarmed:D8041CD" H 10300 2850 50  0001 C CNN
@@
 NoConn ~ 5150 1200
 $Comp
-L Potentiometer_Digital:MCP41010 U2
+L Potentiometer_Digital:MCP41010 U1
 U 1 1 602EE2CA
 P 1400 1200
-F 0 "U2" H 1400 1781 50  0000 C CNN
+F 0 "U1" H 1400 1781 50  0000 C CNN
 F 1 "MCP41010" H 1400 1690 50  0000 C CNN
 F 2 "Package_DIP:DIP-8_W7.62mm" H 1400 1200 50  0001 C CNN
@@
 Text Label 1400 1950 0    50   ~ 0
 GND
+$Comp
+L power:+5V #PWR01
+U 1 1 60E8FE0C
+P 5800 850
+F 0 "#PWR01" H 5800 700 50  0001 C CNN
+F 1 "+5V" H 5815 1023 50  0000 C CNN
+F 2 "" H 5800 850 50  0001 C CNN
+F 3 "" H 5800 850 50  0001 C CNN
+	1    5800 850
+	1    0    0    -1
+$EndComp
+$Comp
+L power:GND #PWR02
+U 1 1 60E90983
+P 5800 1300
+F 0 "#PWR02" H 5800 1050 50  0001 C CNN
+F 1 "GND" H 5805 1127 50  0000 C CNN
+F 2 "" H 5800 1300 50  0001 C CNN
+F 3 "" H 5800 1300 50  0001 C CNN
+	1    5800 1300
+	1    0    0    -1
+$EndComp
+Wire Wire Line
+	5800 850  5800 950
+Wire Wire Line
+	5800 950  6050 950
+Wire Wire Line
+	5800 1300 5800 1150
+Wire Wire Line
+	5800 1150 6050 1150
+Text Label 6050 950  0    50   ~ 0
+VCC
+Text Label 6050 1150 0    50   ~ 0
+GND
 $EndSCHEMATC

Commit message: Add new boards
Parts:
- removed DS1, DS2, DS3, DS4, DS5, DS6, DS7, DS8: D8014CD, Disarmed:D8041CD, symbol DisarmedParts:D8014CD
- removed J1: Conn_02x04_Counter_Clockwise, Connector_PinSocket_2.54mm:PinSocket_2x04_P2.54mm_Vertical, symbol Connector_Generic:Conn_02x04_Counter_Clockwise
- removed U1: MCP41010, Package_DIP:DIP-8_W7.62mm, symbol Potentiometer_Digital:MCP41010
- added C1: 0.1uF, Capacitor_SMD:C_1812_4532Metric_Pad1.57x3.40mm_HandSolder, symbol Device:C
- added C2: 10uF, Capacitor_SMD:C_1812_4532Metric_Pad1.57x3.40mm_HandSolder, symbol Device:C
- added J1: Conn_02x03_Odd_Even, Connector_PinHeader_2.54mm:PinHeader_2x03_P2.54mm_Vertical, symbol Connector_Generic:Conn_02x03_Odd_Even
- added J10, J3, J4, J5, J6, J7, J8, J9: Conn_02x02_Odd_Even, Connector_PinSocket_2.54mm:PinSocket_2x02_P2.54mm_Vertical, symbol Connector_Generic:Conn_02x02_Odd_Even
- added J11, J12, J13, J14: Conn_02x04_Odd_Even, Connector_PinSocket_2.54mm:PinSocket_2x04_P2.54mm_Vertical, symbol Connector_Generic:Conn_02x04_Odd_Even
- added J2: Conn_01x02_Male, Connector_PinHeader_2.54mm:PinHeader_1x02_P2.54mm_Vertical, symbol Connector:Conn_01x02_Male
- added R2, R3, R4: RMIN (2K), Resistor_SMD:R_1210_3225Metric_Pad1.30x2.65mm_HandSolder, symbol Device:R
- added R5: 10K, Resistor_SMD:R_1210_3225Metric_Pad1.30x2.65mm_HandSolder, symbol Device:R
- added RV1, RV2, RV3, RV4: R_POT, 3362P-1-103LF:TRIM_3362P-1-103LF, symbol Device:R_POT
- added U1: ATTINY85-20PU, digikey-footprints:DIP-8_W7.62mm, symbol dk_Embedded-Microcontrollers:ATTINY85-20PU
- R1: value 2k -> RMIN (2K); footprint Resistor_THT:R_Axial_DIN0207_L6.3mm_D2.5mm_P15.24mm_Horizontal -> Resistor_SMD:R_1210_3225Metric_Pad1.30x2.65mm_HandSolder
Connections:
- net labels added: ISET1, ISET2, ISET3, ISET4, MISO_DATA, MOSI_SDA, RST, SCK_SCL
- net labels removed: CCSEL, DATA, ISET
- wire segments 209 -> 205
- no-connect marks 3 -> 5
Other:
- note added: "Drives MAX/MCP chips via SPI like protocol using SPI hardware (or software transfer)"
- note added: "ISP used for programming, shares pins with master system I2C"
- note added: "Implements a I2C interface to the master system."
- moved on the sheet: U2, U3, U4, U5
