File: Disarmed/Switch_Panel.sch (KiCad schematic (older format))
At the start: 55 parts, among them J1 USB_B_Micro, J10 Conn_01x08, J11 Conn_01x04, J2 Conn_01x02_Male, J3 Conn_02x03_Odd_Even, J4 Conn_01x06, J5 Conn_02x06_Counter_Clockwise, J6 Conn_02x06_Counter_Clockwise, J7 Conn_01x08, J8 Conn_01x08, J9 Conn_01x08, SW1 SW_SPST_LED, SW10 SW_SPST, SW11 SW_SPST_LED, SW12 SW_SPST, SW13 SW_SPST, SW14 SW_SPST_LED, SW15 SW_SPST_LED, SW16 SW_SPST_LED, SW2 SW_SPST_LED, SW3 SW_SPST_LED, SW4 SW_SPST_LED, SW5 SW_SPST_LED, SW6 SW_SPST, SW7 SW_SPST, SW8 SW_SPST, SW9 SW_SPST_LED, U1 ATMEGA328PB-AU, U2 MCP41010, U3 MAX7219, U4 MCP23017_SP, U5 MCP23017_SP, U6 MCP23017_SP, Y1 Crystal

Commit message: Add new boards
Changed lines of the file:
@@
 $Descr A3 16535 11693
 encoding utf-8
-Sheet 1 5
+Sheet 4 6
 Title ""
 Date ""
@@
 AR Path="/60061CF4/6043BA9A" Ref="J?"  Part="1"
 AR Path="/6043BA9A" Ref="J3"  Part="1"
-F 0 "J3" H 2550 5317 50  0000 C CNN
+F 0 "J?" H 2550 5317 50  0000 C CNN
 F 1 "Conn_02x03_Odd_Even" H 2550 5226 50  0000 C CNN
 F 2 "Connector_PinHeader_2.54mm:PinHeader_2x03_P2.54mm_Vertical" H 2500 5000 50  0001 C CNN
@@
 AR Path="/60061CF4/6043BAC2" Ref="R?"  Part="1"
 AR Path="/6043BAC2" Ref="R1"  Part="1"
-F 0 "R1" H 1970 8946 50  0000 L CNN
+F 0 "R?" H 1970 8946 50  0000 L CNN
 F 1 "10K" H 1970 8855 50  0000 L CNN
 F 2 "Resistor_SMD:R_1210_3225Metric_Pad1.30x2.65mm_HandSolder" V 1830 8900 50  0001 C CNN
@@
 AR Path="/60061CF4/6043BAD6" Ref="#PWR?"  Part="1"
 AR Path="/6043BAD6" Ref="#PWR02"  Part="1"
-F 0 "#PWR02" H 925 6400 50  0001 C CNN
+F 0 "#PWR?" H 925 6400 50  0001 C CNN
 F 1 "GND" H 930 6477 50  0000 C CNN
 F 2 "" H 925 6650 50  0001 C CNN
@@
 AR Path="/60061CF4/6043BADE" Ref="#PWR?"  Part="1"
 AR Path="/6043BADE" Ref="#PWR01"  Part="1"
-F 0 "#PWR01" H 925 5800 50  0001 C CNN
+F 0 "#PWR?" H 925 5800 50  0001 C CNN
 F 1 "+5V" H 940 6123 50  0000 C CNN
 F 2 "" H 925 5950 50  0001 C CNN
@@
 AR Path="/60061CF4/6043BAE6" Ref="J?"  Part="1"
 AR Path="/6043BAE6" Ref="J2"  Part="1"
-F 0 "J2" H 2583 5631 50  0000 C CNN
+F 0 "J?" H 2583 5631 50  0000 C CNN
 F 1 "Conn_01x02_Male" H 2583 5540 50  0000 C CNN
 F 2 "Connector_PinHeader_2.54mm:PinHeader_1x02_P2.54mm_Vertical" H 2475 5450 50  0001 C CNN
@@
 AR Path="/60061CF4/6045EBA2" Ref="R?"  Part="1"
 AR Path="/6045EBA2" Ref="R9"  Part="1"
-F 0 "R9" V 5643 5325 50  0000 C CNN
+F 0 "R?" V 5643 5325 50  0000 C CNN
 F 1 "2k" V 5734 5325 50  0000 C CNN
 F 2 "Resistor_SMD:R_1210_3225Metric_Pad1.30x2.65mm_HandSolder" V 5780 5325 50  0001 C CNN
@@
 AR Path="/60061CF4/6045EBAA" Ref="U?"  Part="1"
 AR Path="/6045EBAA" Ref="U2"  Part="1"
-F 0 "U2" H 4950 5906 50  0000 C CNN
+F 0 "U?" H 4950 5906 50  0000 C CNN
 F 1 "MCP41010" H 4950 5815 50  0000 C CNN
 F 2 "Package_DIP:DIP-8_W7.62mm" H 4950 5325 50  0001 C CNN
@@
 AR Path="/60061CF4/6043BAAE" Ref="C?"  Part="1"
 AR Path="/6043BAAE" Ref="C4"  Part="1"
-F 0 "C4" H 4090 9446 50  0000 L CNN
+F 0 "C?" H 4090 9446 50  0000 L CNN
 F 1 "0.1uF" H 4090 9355 50  0000 L CNN
 F 2 "Capacitor_SMD:C_1812_4532Metric_Pad1.57x3.40mm_HandSolder" H 4013 9250 50  0001 C CNN
